Commit message: interfaz_dos_piernas

File: ros2_ws/src/robot_description/urdf/Pata_Robo_Parcial_URDF_V1.2.urdf (robot description, URDF)
Before this commit: robot Pata_Robo_Parcial_URDF_V1.2, 4 links, 3 joints
Links:
- added link world
Joints:
- added joint world_to_base: type fixed, parent world, child Base_link, origin xyz=0 0 1.008062 rpy=0 1.57079632679 0
