Commit message: Separar URDF por pata (der/izq), arreglar rodilla invertida y reordenar limites
- robot_description: URDF/xacro independientes por pierna (urdf_der/urdf_izq),
  mallas por pata, mesh paths y colores corregidos, joint duplicado eliminado,
  eje de rodilla invertido corregido en ambas piernas.
- robot_bringup y robot_description: launch files por pata (der/izq) en vez
  de uno solo generico.
- robot_control/robot_teleop: el limite interno (control_node) y el limite
  visual del slider (teleop_node) ya no se pasan desde los launch, viven cada
  uno en su propio nodo.
- ARCHITECTURE.md actualizado a la nueva arquitectura de dos patas.
- servo_params.h: calibracion de OSC_FREQ_HZ del PCA9685.

Co-Authored-By: Claude Sonnet 5 <noreply@anthropic.com>

File: ros2_ws/src/robot_description/urdf/urdf_izq/Pata_Izq_Robo_Parcial_URDF_V2.5.urdf (robot description, URDF)
Before this commit: robot Pata_Robo_Parcial_URDF_V1.2, 5 links, 4 joints
Links:
- removed link Ankle_Link
- removed link Hip_Link
- removed link Knee_Link
- removed link world
- added link Left_Hip_Pitch_Link, mass 0.21755; collision mesh filename=package://robot_description/meshes/meshes_izq/Left_Hip_Pitc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; visual mesh filename=package://robot_description/meshes/meshes_izq/Left_Hip_Pitc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
- added link Left_Hip_Roll_Link, mass 0.19411; collision mesh filename=package://robot_description/meshes/meshes_izq/Left_Hip_Roll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; visual mesh filename=package://robot_description/meshes/meshes_izq/Left_Hip_Roll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
- added link Left_Knee_Link, mass 0.38813; collision mesh filename=package://robot_description/meshes/meshes_izq/Left_Knee_Lin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; visual mesh filename=package://robot_description/meshes/meshes_izq/Left_Knee_Lin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
- link Base_link: mass 26.056 -> 25.798; geometry collision mesh filename=package://robot_description/meshes/meshes_izq/Base_link.STL; visual mesh filename=package://robot_description/meshes/meshes_izq/Base_link.STL
Joints:
- removed joint Ankle_Joint
- removed joint Hip_Joint
- removed joint Knee_Joint
- removed joint world_to_base
- added joint Left_Hip_Pitch_Joint: type revolute, parent Left_Hip_Roll_Link, child Left_Hip_Pitch_Link, origin xyz=0.11885 0 0 rpy=-1.5708 0 0, axis 0 0 1, limit lower=-2.0071 upper=2.0071 effort=100 velocity=100
- added joint Left_Hip_Roll_Joint: type revolute, parent Base_link, child Left_Hip_Roll_Link, origin xyz=0.083749 0 -0.2004 rpy=1.5708 0 0, axis 0 0 -1, limit lower=-0.34907 upper=2.2689 effort=100 velocity=100
- added joint Left_Knee_Joint: type revolute, parent Left_Hip_Pitch_Link, child Left_Knee_Link, origin xyz=0.23605 0 0 rpy=3.1416 0 0, axis 0 0 -1, limit lower=-2.0071 upper=2.0071 effort=100 velocity=100
