Commit message: Correción del sistema de referencia fijo en (Base_link), modificación de codigos de cinematica.

File: ros2_ws/src/robot_description/urdf/urdf_completo/Pata_Pacial2URDFV9.urdf (robot description, URDF)
Before this commit: robot Pata_Pacial2URDFV6, 7 links, 6 joints
Joints:
- joint Left_Hip_Roll_Joint: limit lower=-0.34907 upper=1.5708 effort=100 velocity=100 -> lower=0 upper=1.5708 effort=100 velocity=100; origin xyz=0.078873 -0.10909 -0.14579 rpy=3.1416 -1.5708 0 -> xyz=0.10909 0.078873 -0.14579 rpy=4.7124 -1.5708 0
- joint Left_Knee_Joint: origin xyz=0 0.313239999999995 -0.000121751528806113 rpy=0 0 0 -> xyz=0 0.31324 -0.00012175 rpy=0 0 0
- joint Right_Hip_Roll_Joint: limit lower=-0.34907 upper=1.5708 effort=100 velocity=100 -> lower=0 upper=1.5708 effort=100 velocity=100; origin xyz=0.065472 -0.10907 0.14406 rpy=3.1416 -1.5708 0 -> xyz=0.10907 0.065472 0.14406 rpy=4.7124 -1.5708 0

File: ros2_ws/src/robot_description/urdf/urdf_completo/robot_completo.urdf.xacro (robot description, xacro)
@@ -2,10 +2,15 @@
 <robot name="robot_completo" xmlns:xacro="http://www.ros.org/wiki/xacro">
   <!--
-    Wrapper xacro para el robot completo (Pata_Pacial2URDFV6: ambas patas
-    sobre el mismo Base_link). El CAD fue exportado con el eje +Y hacia
-    arriba (las patas cuelgan hacia -Y y se separan sobre Z); esta rotacion
-    de +90 grados en X lo deja vertical en RViz, con +Y del CAD -> +Z del
-    mundo y la pata derecha hacia -Y del mundo, sin cambiar la cinematica
-    ni los ejes de las articulaciones.
+    Wrapper xacro para el robot completo (Pata_Pacial2URDFV9: ambas patas
+    sobre el mismo Base_link). En V9 el Base_link del CAD tiene los mismos
+    ejes que la base {0} de la cinemática (cinematica_directa_der_izq.py):
+      +X  a lo largo de la pierna, hacia ABAJO
+      +Y  adelante / atrás
+      +Z  lateral (pata izquierda hacia -Z, derecha hacia +Z)
+    Esta rotación (rpy = 0, +90°, -90°) lo deja vertical en RViz:
+      +X Base_link -> -Z mundo  (las patas cuelgan)
+      +Y Base_link -> +X mundo
+      +Z Base_link -> -Y mundo  (pata izquierda hacia +Y del mundo)
+    sin cambiar la cinemática ni los ejes de las articulaciones.
   -->
   <link name="world" />
@@ -13,6 +18,6 @@
     <parent link="world" />
     <child link="Base_link" />
-    <origin xyz="0 0 0" rpy="1.57079632679 0 0" />
+    <origin xyz="0 0 0" rpy="0 1.57079632679 -1.57079632679" />
   </joint>
-  <xacro:include filename="$(find robot_description)/urdf/urdf_completo/Pata_Pacial2URDFV6.urdf" />
+  <xacro:include filename="$(find robot_description)/urdf/urdf_completo/Pata_Pacial2URDFV9.urdf" />
 </robot>
